Commit message: this seems to run half-way decently

File: res/scenario_1/panda_US.urdf (robot description, URDF)
Before this commit: robot panda_US, 8 links, 7 joints
Links:
- removed link base_link
- removed link link1
- removed link link2
- removed link link3
- removed link link4
- removed link link5
- removed link link6
- removed link link7
- added link panda_link0, mass 2.92; collision mesh filename=/home/lovis/RUSRes/CollisionAvoidance/robot/meshes/panda/co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; visual mesh filename=/home/lovis/RUSRes/CollisionAvoidance/robot/meshes/panda/vi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
- added link panda_link1, mass 2.74; collision mesh filename=/home/lovis/RUSRes/CollisionAvoidance/robot/meshes/panda/co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; visual mesh filename=/home/lovis/RUSRes/CollisionAvoidance/robot/meshes/panda/vi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
- added link panda_link2, mass 2.74; collision mesh filename=/home/lovis/RUSRes/CollisionAvoidance/robot/meshes/panda/co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; visual mesh filename=/home/lovis/RUSRes/CollisionAvoidance/robot/meshes/panda/vi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
- added link panda_link3, mass 2.38; collision mesh filename=/home/lovis/RUSRes/CollisionAvoidance/robot/meshes/panda/co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; visual mesh filename=/home/lovis/RUSRes/CollisionAvoidance/robot/meshes/panda/vi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
- added link panda_link4, mass 2.38; collision mesh filename=/home/lovis/RUSRes/CollisionAvoidance/robot/meshes/panda/co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; visual mesh filename=/home/lovis/RUSRes/CollisionAvoidance/robot/meshes/panda/vi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
- added link panda_link5, mass 2.74; collision mesh filename=/home/lovis/RUSRes/CollisionAvoidance/robot/meshes/panda/co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; visual mesh filename=/home/lovis/RUSRes/CollisionAvoidance/robot/meshes/panda/vi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
- added link panda_link6, mass 1.55; collision mesh filename=/home/lovis/RUSRes/CollisionAvoidance/robot/meshes/panda/co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; visual mesh filename=/home/lovis/RUSRes/CollisionAvoidance/robot/meshes/panda/vi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
- added link panda_link7, mass 0.54; collision mesh filename=/home/lovis/RUSRes/CollisionAvoidance/robot/meshes/panda/co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; visual mesh filename=/home/lovis/RUSRes/CollisionAvoidance/robot/meshes/panda/vi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
- added link us_image; visual mesh filename=
- added link us_probe, mass 0.73; collision mesh filename=/home/lovis/RUSRes/CollisionAvoidance/robot/meshes/panda/vi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; visual mesh filename=/home/lovis/RUSRes/CollisionAvoidance/robot/meshes/panda/vi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
- added link us_pump, mass 0.0; collision mesh filename=/home/lovis/RUSRes/CollisionAvoidance/robot/meshes/panda/vi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; visual mesh filename=/home/lovis/RUSRes/CollisionAvoidance/robot/meshes/panda/vi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
- added link world
Joints:
- removed joint joint1
- removed joint joint2
- removed joint joint3
- removed joint joint4
- removed joint joint5
- removed joint joint6
- removed joint joint7
- added joint panda_joint1: type revolute, parent panda_link0, child panda_link1, origin xyz=0 0 0.333 rpy=0 0 0, axis 0 0 1, limit lower=-2.7973 upper=2.7973 effort=87 velocity=2.1750
- added joint panda_joint10: type fixed, parent us_pump, child us_image, origin xyz=0 0.147470000000000 0.028990000000000 rpy=-1.57079632679 0 -3.14159265359
- added joint panda_joint2: type revolute, parent panda_link1, child panda_link2, origin xyz=0 0 0 rpy=-1.57079632679 0 0, axis 0 0 1, limit lower=-1.6628 upper=1.6628 effort=87 velocity=2.1750
- added joint panda_joint3: type revolute, parent panda_link2, child panda_link3, origin xyz=0 -0.316 0 rpy=1.57079632679 0 0, axis 0 0 1, limit lower=-2.7973 upper=2.7973 effort=87 velocity=2.1750
- added joint panda_joint4: type revolute, parent panda_link3, child panda_link4, origin xyz=0.0825 0 0 rpy=1.57079632679 0 0, axis 0 0 1, limit lower=-2.9718 upper=0.1698 effort=87 velocity=2.1750
- added joint panda_joint5: type revolute, parent panda_link4, child panda_link5, origin xyz=-0.0825 0.384 0 rpy=-1.57079632679 0 0, axis 0 0 1, limit lower=-2.7973 upper=2.7973 effort=12 velocity=2.6100
- added joint panda_joint6: type revolute, parent panda_link5, child panda_link6, origin xyz=0 0 0 rpy=1.57079632679 0 0, axis 0 0 1, limit lower=-0.0175 upper=3.6525 effort=12 velocity=2.6100
- added joint panda_joint7: type revolute, parent panda_link6, child panda_link7, origin xyz=0.088 0 0 rpy=1.57079632679 0 0, axis 0 0 1, limit lower=-2.7973 upper=2.7973 effort=12 velocity=2.6100
- added joint panda_joint8: type fixed, parent panda_link7, child us_probe, origin xyz=0 0 0.107 rpy=0 0 0, axis 0 0 0
- added joint panda_joint9: type fixed, parent us_probe, child us_pump, origin xyz=0 0 0.0 rpy=0 0 0, axis 0 0 0
- added joint panda_joint_world: type fixed, parent world, child panda_link0, origin xyz=0 0 0 rpy=0 0 0
